Commit message: Remove manual_grasp_link

File: macros/tools/robotiq_2f_85.xacro (robot description, xacro)
@@ -14,4 +14,5 @@
       <origin xyz="0 0 0" rpy="0 0 0"/>
     </xacro:robotiq_gripper>
+    <!-- We use grasp_link frame to perform quick tasks such as inspect surface -->
     <link name="grasp_link"/>
     <joint name="grasp_link_joint" type="fixed">
@@ -20,11 +21,4 @@
       <origin xyz="0.0 0.0 0.134" rpy="0.0 0.0 ${pi}"/>
     </joint>
-    <!-- Moveit Studio requires a link name called manual_grasp_link to perform quick tasks such as inspect surface -->
-    <link name="manual_grasp_link"/>
-    <joint name="manual_grasp_joint" type="fixed">
-      <parent link="grasp_link"/>
-      <child link="manual_grasp_link"/>
-      <origin xyz="0 0 0" rpy="${pi / 180.0 * 5} 0 0"/>
-    </joint>
   </xacro:macro>
 </robot>
