Commit message: Add closed ceiling collision for space station

File: descriptions/furniture/space_station/space_station.urdf.xacro (robot description, xacro)
@@ -10,14 +10,24 @@
     <link name="space_station">
       <visual>
-          <origin xyz="0 0 0" rpy="0 0 0"/>
-          <geometry>
-              <mesh filename="package://picknik_accessories/descriptions/furniture/space_station/space_booth.dae"/>
-          </geometry>
+        <origin xyz="0 0 0" rpy="0 0 0"/>
+        <geometry>
+          <mesh filename="package://picknik_accessories/descriptions/furniture/space_station/space_booth.dae"/>
+        </geometry>
       </visual>
       <collision>
         <origin xyz="0 0 0" rpy="0 0 0"/>
-          <geometry>
-              <mesh filename="package://picknik_accessories/descriptions/furniture/space_station/space_booth.dae"/>
-          </geometry>
+        <geometry>
+          <mesh filename="package://picknik_accessories/descriptions/furniture/space_station/space_booth.dae"/>
+        </geometry>
+      </collision>
+      <!-- box collision for the ceiling so that the robot does not try to plan into the open gaps of the ceiling -->
+      <collision>
+        <origin xyz="0 0 2.325" rpy="0 0 0"/>
+        <geometry>
+          <box size="3 2.1 0.05"/>
+        </geometry>
+        <material>
+          <color rgba="1.0 0 0 1"/>
+        </material>
       </collision>
       <inertial>

Commit message: make collision thicker so robot doesn't come as close to the ceiling

File: descriptions/furniture/space_station/space_station.urdf.xacro (robot description, xacro)
@@ -23,7 +23,7 @@
       <!-- box collision for the ceiling so that the robot does not try to plan into the open gaps of the ceiling -->
       <collision>
-        <origin xyz="0 0 2.325" rpy="0 0 0"/>
+        <origin xyz="0 0 2.3" rpy="0 0 0"/>
         <geometry>
-          <box size="3 2.1 0.05"/>
+          <box size="3 2.1 0.08"/>
         </geometry>
         <material>

Commit message: Make space station ceiling thicker

File: descriptions/furniture/space_station/space_station.urdf.xacro (robot description, xacro)
@@ -25,5 +25,5 @@
         <origin xyz="0 0 2.3" rpy="0 0 0"/>
         <geometry>
-          <box size="3 2.1 0.08"/>
+          <box size="3 2.1 0.14"/>
         </geometry>
         <material>
